File: pcb/CA80.kicad_pcb (KiCad board)
At the start: 4 copper layers, 160 x 124 mm, 96 parts, among them J1 Jumper_3_Bridged12, J10 Conn_01x03_Socket, J2 Jumper_3_Bridged12, J27 Conn_01x06_Socket, J3 Jumper_3_Bridged12, J36 Conn_02x07_Odd_Even, J4 Conn_01x05_Socket, J5 Jumper_3_Bridged12, J6 Conn_02x04_Odd_Even, J7 Conn_01x04_Socket, J8 Conn_01x06_Socket, J9 Conn_01x06_Socket, T1 BC557, U1 7400, U10 2764, U11 2764, U12 2764, U13 74LS132, U14 LM741, U15 74LS123, U16 74LS138, U2 7400, U20 74LS42, U21 8255A, U22 Z80A_CTC, U23 74LS06, U24 74LS06, U25 74LS06, U3 7493, U4 74LS138, U5 4518, U6 4518, U7 8255A, U8 Z80CPU, U9 2764

Commit message: update
Routing:
- net /A11: track 115.3 -> 116.5 mm
- net /A13: track 117.0 -> 118.1 mm
- net /A14: track 146.6 -> 147.4 mm
- net /D3: track 229.6 -> 228.9 mm
